File: Hardware/KiCad9/cloudSmoker_ver2b.kicad_sch (KiCad schematic)
At the start: 52 parts, among them J1 AudioJack2_SwitchT, J10 Conn_01x02_Pin, J11 Conn_01x02_Pin, J12 Conn_01x02_Pin, J2 AudioJack2_SwitchT, J3 AudioJack2_SwitchT, J4 AudioJack2_SwitchT, J5 Conn_01x02_Pin, J6 Conn_01x02_Pin, J7 Conn_01x02_Pin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

Commit message: kicad updates
Parts:
- added LED4: Yellow, JLCImport:FC-1608YXK-585F08, symbol Device:LED_Small
- added R15: 100, JLCImport:0603WAF1000T5E, symbol Device:R
Connections:
- net +3.3V: now also U3.6 (IO7), R15.1
- net GND: now also LED4.1 (K)
- net at Q2.2 (S), R12.2: now also U3.5 (IO6); no longer SW2.2, U3.8 (IO9)
- net at Q1.2 (S), R11.2: now also U3.4 (IO5); no longer U3.7 (IO8)
- net DEBUG_RX: now reaches U3.11 (IO20/RXD)
- net DEBUG_TX: now reaches U3.12 (IO21/TXD)
- new net: LED4.2 (A), R15.2
- new net ~{Boot}: SW2.2, U3.8 (IO9)
- no-connect marks 9 -> 12
Other:
- note added: "boot"
- moved on the sheet: C1, C2, C3, C4, LED1, LED2, Q1, Q2, R11, R12, R13, R14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
