File: Hardware/KiCad9/cloudSmoker_ver2d.kicad_sch (KiCad schematic)
At the start: 67 parts, among them J1 AudioJack2_SwitchT, J10 Conn_01x02_Pin, J11 Conn_01x02_Pin, J12 Conn_01x05, J13 Conn_01x08, J2 AudioJack2_SwitchT, J3 AudioJack2_SwitchT, J4 AudioJack2_SwitchT, J5 Conn_01x04_Pin, J6 Conn_01x04_Pin, J7 Conn_01x02_Pin, J8 Conn_01x02_Pin, J9 Conn_01x02_Pin, Q1 BSS138, Q2 BSS138, SW1 TS-1088-AR02016, SW2 TS-1088-AR02016, SW3 RotaryEncoder_Switch, U1 GT-USB-7010ASV, U2 SRV05-4-P-T7, U3 TLV76733DGNR, U4 SRV05-4-P-T7, U5 ESP32-C3-WROOM-02U-N4, U6 ADS1115IRUGR, U7 INA226AIDGSR

Commit message: update board files for v2d
Parts:
- removed C10: 10uF, JLCImport:CL10A106MA8NRNC, symbol Device:C
- removed C11: 100nF, JLCImport:CC0603KRX7R9BB104, symbol Device:C
- removed C12: 1uF, JLCImport:CC0603KRX7R9BB104, symbol Device:C
- removed R5, R9: 10k, JLCImport:0603WAF1002T5E, symbol Device:R
- removed SW1, SW2: TS-1088-AR02016, JLCImport:TS-1088-AR02016, symbol Switch:SW_Push
- removed U3: TLV76733DGNR, JLCImport:TLV76733DGNR, symbol JLCImport:TLV76733DGNR
- added C4: 10uF, JLCImport:CL21A106KAYNNNE, symbol Device:C
- added C6: 100nF, JLCImport:CC0603KRX7R9BB104, symbol Device:C
- added C7: 1uF, JLCImport:CC0603KRX7R9BB104, symbol Device:C
- added H5, H6: M3, MountingHole:MountingHole_3.2mm_M3, symbol Mechanical:MountingHole
- added J2, J5: Conn_01x04_Socket, symbol Connector:Conn_01x04_Socket
- added J8: Conn_01x05_Socket, symbol Connector:Conn_01x05_Socket
- added JP1, JP2, JP3: SolderJumper_2_Bridged, Jumper:SolderJumper-2_P1.3mm_Bridged_RoundedPad1.0x1.5mm, symbol Jumper:SolderJumper_2_Bridged
- added R10, R11, R12, R8: 22, JLCImport:PTFR0603B120KP9, symbol Device:R
- added R16: 10k, JLCImport:0603WAF1002T5E, symbol Device:R
- added R17, R19: 5.1k, JLCImport:0603WAF5101T5E, symbol Device:R
- added R6, R7: 10, JLCImport:PTFR0603B120KP9, symbol Device:R
- added SW2, SW3: SW_Push_Dual, JLCImport:TS-1187A-B-A-B, symbol Switch:SW_Push_Dual
- added TP1: TP_GND_Clip, TestPoint:TestPoint_Bridge_Pitch5.08mm_Drill0.7mm, symbol Connector:TestPoint
- added TP10: TP_Pit, TestPoint:TestPoint_Pad_D1.0mm, symbol Connector:TestPoint
- added TP11: TP_Meat1, TestPoint:TestPoint_Pad_D1.0mm, symbol Connector:TestPoint
- added TP12: TP_AGND, TestPoint:TestPoint_Pad_D1.0mm, symbol Connector:TestPoint
- added TP13: TP_Meat2, TestPoint:TestPoint_Pad_D1.0mm, symbol Connector:TestPoint
- added TP14: TP_Meat3, TestPoint:TestPoint_Pad_D1.0mm, symbol Connector:TestPoint
- added TP2: TP_3V3, TestPoint:TestPoint_Pad_D1.0mm, symbol Connector:TestPoint
- added TP3, TP6, TP9: TP_GND, TestPoint:TestPoint_Pad_D1.0mm, symbol Connector:TestPoint
- added TP4: TP_EN, TestPoint:TestPoint_Pad_D1.0mm, symbol Connector:TestPoint
- added TP5: TP_5V, TestPoint:TestPoint_Pad_D1.0mm, symbol Connector:TestPoint
- added TP7: TP_SPI_SCK, TestPoint:TestPoint_Pad_D1.0mm, symbol Connector:TestPoint
- added TP8: TP_GIO9, TestPoint:TestPoint_Pad_D1.0mm, symbol Connector:TestPoint
- added U1: TLV76733DGNR, JLCImport:TLV76733DGNR, symbol JLCImport:TLV76733DGNR
- FID1, FID2, FID3: footprint (none) -> Fiducial:Fiducial_1mm_Mask2mm
- H1, H2, H3, H4: footprint (none) -> MountingHole:MountingHole_3.2mm_M3_Pad_Via
- J10: renamed from J5; symbol Connector_Generic:Conn_01x04 -> Connector:Conn_01x04_Socket
- J11: renamed from J7; value Conn_01x02_Pin -> Conn_01x04_Pin
- J14: renamed from J6; symbol Connector_Generic:Conn_01x04 -> Connector:Conn_01x04_Socket
- J15: renamed from J8; value Conn_01x02_Pin -> Conn_01x04_Pin
- J3: renamed from J10; value Conn_01x02_Pin -> Conn_01x04_Pin
- J6: renamed from J11; value Conn_01x02_Pin -> Conn_01x04_Pin
- J7: renamed from J12; footprint (none) -> Connector_JST:JST_XH_B5B-XH-A_1x05_P2.50mm_Vertical
- Q1, Q2: footprint Package_TO_SOT_SMD:SOT-23 -> JLCImport:BSS138_C7420339
- R13: renamed from R17; symbol Device:R_Shunt -> Device:R
- R14: value 10k -> 22; footprint JLCImport:0603WAF1002T5E -> JLCImport:PTFR0603B120KP9; LCSC C25804 -> C23345; Manufacturer Part 0603WAF1002T5E -> 0603WAF220JT5E
- U2: renamed from U1; footprint JLCImport:GT-USB-7010ASV -> Connector_USB:USB_C_Receptacle_G-Switch_GT-USB-7010ASV
- U3: renamed from U7; footprint Package_SO:VSSOP-10_3x3mm_P0.5mm -> JLCImport:INA226AIDGSR
- U4: renamed from U5; footprint RF_Module:ESP32-C3-WROOM-02U -> JLCImport:ESP32-C3-WROOM-02U-N4
- U5: renamed from U2; footprint Package_TO_SOT_SMD:SOT-23-6 -> JLCImport:SRV05-4-P-T7
- U6: footprint Package_SO:TSSOP-10_3x3mm_P0.5mm -> JLCImport:ADS1115IRUGR
- U7: renamed from U4; footprint Package_TO_SOT_SMD:SOT-23-6 -> JLCImport:SRV05-4-P-T7
- renumbered C7 to C10, C8 to C11, C9 to C3, C13 to C5, C5 to C8, C6 to C9, J9 to J1, J2 to J12, J3 to J13, J4 to J16, J13 to J4, J1 to J9, R3 to R1, R4 to R18, R10 to R2, R7 to R20, R6 to R21, R8 to R22, R11 to R23, R12 to R24, R1 to R3, R2 to R4, R13 to R5, R16 to R9, SW3 to SW1
Connections:
- net +3.3V: now also J7.5 (Pin_5), C4.1, R16.2, R17.2, R19.2, TP2.1, U1.1 (OUT), U1.2 (SNS); no longer R14.2
- net +5V: now also C1.1, R1.1, R13.2, C6.2, R7.1, TP5.1, U1.5 (EN), U1.8 (IN); no longer J7.5 (Pin_5), R13.4
- net DISP_BL: now also U4.4 (IO5); no longer U4.18 (IO0)
- net DISP_CS: now also R9.2, R12.1; no longer U4.10 (IO10)
- net DISP_DC: now also R8.1; no longer R9.2, U4.7 (IO8)
- net ENC_CLK: now also U4.15 (IO3); no longer U4.3 (IO4)
- net ENC_DT: now also U4.16 (IO2); no longer U4.4 (IO5)
- net ENC_SW: now also U4.10 (IO10); no longer U4.17 (IO1)
- net GND: now also C4.2, C7.2, JP1.1 (A), JP2.2 (B), JP3.2 (B), SW2.3, SW2.4, SW3.3, SW3.4, TP1.1, TP12.1, TP3.1, TP6.1, TP9.1, U1.4 (GND), U1.6 (GND), U1.9 (EP); no longer LED1.1 (K), LED2.1 (K), LED3.1 (K)
- net MEAT1: now also TP11.1
- net MEAT2: now also TP13.1
- net MEAT3: now also TP14.1
- net PIT: now also TP10.1
- net SPI_MOSI: now also R11.2; no longer U4.6 (IO7)
- net SPI_SCK: now also R10.1, TP7.1; no longer U4.5 (IO6)
- net USB_D+: now also U5.6 (IO4); no longer U5.3 (IO2)
- net VBUS: now also C6.1, R6.1; no longer C1.1, R1.1
- net ~{BOOT}_DISP_RST: now also R14.2, R15.1, SW2.1, SW2.2, TP8.1; no longer R14.1, U4.8 (IO9)
- net ~{RESET}: now also C7.1, R16.1, SW3.1, SW3.2, TP4.1; no longer R15.1
- net at R3.1, U2.A5 (CC1): now also U5.3 (IO2)
- net at R4.1, U2.B5 (CC2): now also U5.4 (IO3)
- net MEAT1_IN: now reaches J11.4 (Pin_4), PR2.2, R22.2, U7.3 (IO2)
- net PIT_IN: now reaches J11.2 (Pin_2), PR1.2, R21.2, U7.1 (IO1)
- net MEAT2_IN: now reaches J15.2 (Pin_2), PR3.2, R23.2, U7.4 (IO3)
- net Supply: now reaches U3.10 (Vin+)
- net Supply: now also R6.2; no longer R13.2
- net Load: now reaches U3.9 (Vin-)
- net Load: now also R7.2; no longer R13.3
- net MEAT3_IN: now reaches J15.4 (Pin_4), PR4.2, R24.2, U7.6 (IO4)
- net at J4.1 (Pin_1): now also J5.4 (Pin_4)
- net at J4.2 (Pin_2): now also J5.3 (Pin_3)
- net at J4.3 (Pin_3): now also J5.2 (Pin_2)
- net at J4.4 (Pin_4): now also J5.1 (Pin_1)
- net at J4.5 (Pin_5): now also J2.4 (Pin_4)
- net at J4.6 (Pin_6): now also J2.3 (Pin_3)
- net at J4.7 (Pin_7): now also J2.2 (Pin_2)
- net at J4.8 (Pin_8): now also J2.1 (Pin_1)
- net SCL_3V3 renamed I2C_SCL_3V3
- net I2C_SCL_3V3: now also U3.5 (SCL), U4.17 (IO1), R19.1
- net SCL_5V renamed I2C_SCL_5V
- removed net SDA_3V3: Q1.2 (S), U3.4 (SDA), U3.5 (SCL), U4.15 (IO3), U4.16 (IO2)
- net SDA_5V renamed I2C_SDA_5V
- new net: R12.2, U4.7 (IO8)
- new net: JP3.1 (A), LED3.1 (K)
- new net: R14.1, U4.8 (IO9)
- new net: R8.2, U4.3 (IO4)
- new net: R10.2, U4.5 (IO6)
- new net: R11.1, U4.6 (IO7)
- new net: JP2.1 (A), LED2.1 (K)
- new net: JP1.2 (B), LED1.1 (K)
- new net I2C_SDA_3V3: Q1.2 (S), R17.1, U3.4 (SDA), U4.18 (IO0)
- no-connect marks 39 -> 34
Other:
- note added: "CC lines not usually surge protected but I have 2 free channels in SRV05"
- note added: "Display Headers 2x JST XH 4-pin Male (DNP -add post-fabrication)"
- note added: "Encoder Header JST XH 4-pin Male (DNP -add post-fabrication)"
- note added: "Encoder Header JST XH 5-pin Male (DNP -add post-fabrication)"
- note added: "Ground clip - place on board edge for voltage probing"
- note added: "JST XH 4-pin Female 2.50mm pitch"
- note added: "JST XH 4-pin Male (DNP -add post-fabrication)"
- note added: "JST XH 5-pin Female 2.50mm pitch"
- note added: "Keep high-impedance thermistor traces at least 2-3mm away from mounting holes to avoid metal screw coupling"
- note added: "Kelvin connections required refer to INA226 datasheet"
- note added: "Manually place fiducials to protect artwork"
- note added: "Place ESD Protection close to JST-XH headers to thermistor jacks"
- note added: "Place damping resistors next to pins"
- note added: "Slave Addrsss: 0b1000000 / 0x40"
- note added: "Slave Addrsss: 0b1001000 / 0x48"
- note added: "Test Points on bottom layer"
- note added: "Test Points on bottom layer except TP_SPI_SCK which should be L1 close to pin with nearby ground"
- note added: "UART Header (debug)"
- note added: "VSS=3V3 in order to keep I2C pin voltages ESP32 compliant (otherwise must level shift)"
- note added: "Zip-tie holes for U.Fl antenna strain relief Center-to-Center: 6.0mm Place holes 12-15mm away from U.FL connector Silkscreen: ANT_TIE"
- note removed: "Display Header JST-XH"
- note removed: "Encoder Header JST-XH"
- note removed: "JST XH 4-pin Female (DNP - will add post-fabrication)"
- note removed: "JST XH 4-pin Male"
- note removed: "Place ESD Protection close to JST-XH headers"
- note removed: "Reset Switch"
- note removed: "Slave Addrsss: 1000000b"
- note removed: "Slave Addrsss: 1001000b"
- note removed: "UART / Debug Header (JST-XH)"
- moved on the sheet: C1, C2, C3, FID1, FID2, FID3, J1, J11, J15, J4, J7, LED1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
