File: Hardware/KiCad9/cloudSmoker_ver2e.kicad_sch (KiCad schematic)
At the start: 96 parts, among them J1 Conn_01x02_Pin, J10 Conn_01x04_Pin, J11 Conn_01x04_Pin, J12 AudioJack2_SwitchT, J13 AudioJack2_SwitchT, J14 Conn_01x04_Pin, J15 Conn_01x04_Pin, J16 AudioJack2_SwitchT, J2 Conn_01x04_Socket, J3 Conn_01x04_Pin, J4 Conn_01x08, J5 Conn_01x04_Socket, J6 Conn_01x04_Pin, J7 Conn_01x05, J8 Conn_01x05_Socket, J9 AudioJack2_SwitchT, Q1 BSS138, Q2 BSS138, SW1 RotaryEncoder_Switch, SW2 SW_Push_Dual, SW3 SW_Push_Dual, U1 TLV76733DGNR, U2 GT-USB-7010ASV, U3 INA226AIDGSR, U4 ESP32-C3-WROOM-02U-N4, U5 SRV05-4-P-T7, U6 ADS1115IRUGR, U7 SRV05-4-P-T7

Commit message: update hardware files for version 2e
Parts:
- removed JP3: SolderJumper_2_Bridged, Jumper:SolderJumper-2_P1.3mm_Bridged_RoundedPad1.0x1.5mm, symbol Jumper:SolderJumper_2_Bridged
- added C4, C5: 470nF, JLCImport:CC0603KRX7R9BB104, symbol Device:C
- added R3: 0 ohm, JLCImport:PTFR0603B120KP9, symbol Device:R
- renumbered C8 to C10, C9 to C11, C10 to C12, C11 to C13, C5 to C3, C3 to C7, C4 to C8, C7 to C9, R8 to R10, R9 to R11, R10 to R12, R11 to R13, R12 to R14, R14 to R15, R15 to R16, R16 to R17, R17 to R18, R18 to R19, R19 to R20, R20 to R21, R21 to R22, R22 to R23, R23 to R24, R24 to R25, R6 to R4, R7 to R5, R3 to R6, R4 to R7, R13 to R8, R5 to R9, TP5 to TP1, TP1 to TP2, TP6 to TP3, TP2 to TP4, TP3 to TP5, TP4 to TP6, U3 to U2, U2 to U3
Connections:
- net +5V: no longer U5.5 (VP)
- net DISP_CS: now also R14.2, U4.7 (IO8)
- net GND: now also LED3.1 (K), C4.2, C5.2
- net VBUS: now also U5.5 (VP), C4.1, C5.1, R3.1, R3.2
- net at R6.1, U3.A5 (CC1): no longer U5.3 (IO2)
- net at R7.1, U3.B5 (CC2): no longer U5.4 (IO3)
- no-connect marks 34 -> 36
Other:
- note added: "Ground clip place on board edge for voltage probing"
- note added: "Pi filter Mainly placeholder but trying to get into good habits (per Phil's Lab)"
- note added: "Place pull-ups and damping resistors near pins order: pin -> pull-up (if present) -> damping -> signal"
- note added: "Solder bridge cut to reduce LED power draw"
- note added: "check TP8 is this correct?"
- note removed: "CC lines not usually surge protected but I have 2 free channels in SRV05"
- note removed: "Ground clip - place on board edge for voltage probing"
- note removed: "Place damping resistors next to pins"
- moved on the sheet: C1, C10, C11, C12, C2, C3, C6, J1, JP1, JP2, LED1, LED2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
