File: Hardware/KiCad9/cloudSmoker_ver2f.kicad_sch (KiCad schematic)
At the start: 98 parts, among them J1 Conn_01x02_Pin, J10 Conn_01x04_Pin, J11 Conn_01x04_Pin, J12 AudioJack2_SwitchT, J13 AudioJack2_SwitchT, J14 Conn_01x04_Pin, J15 Conn_01x04_Pin, J16 AudioJack2_SwitchT, J2 Conn_01x04_Socket, J3 Conn_01x04_Pin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

Commit message: update hardware files for cloudSmoker_ver2f
Parts:
- C9: footprint JLCImport:CC0603KRX7R9BB104 -> JLCImport:CL10A105KB8NNNC; LCSC C14663 -> C15849; Manufacturer YAGEO -> Samsung Electro-Mechanics; Manufacturer Part CC0603KRX7R9BB104 -> CL10A105KB8NNNC
- R10, R12, R13, R14, R15: footprint JLCImport:PTFR0603B120KP9 -> JLCImport:R0603_part-C23345
- R3: footprint JLCImport:PTFR0603B120KP9 -> JLCImport:R0603_part-C21189_0-ohm
- R4, R6: footprint JLCImport:PTFR0603B120KP9 -> JLCImport:R0603_part-C22859_10-ohm; LCSC (none) -> C22859; Manufacturer (none) -> UNI-ROYAL(Uniroyal Elec); Manufacturer Part (none) -> 0603WAF100JT5E
- TP1, TP10, TP11, TP12, TP13, TP14, TP2, TP3, TP4, TP5, TP6, TP7, TP8, TP9: now left out of the parts list
Connections:
- net +5V: now also R6.1; no longer R6.2
- net Load: now also R6.2; no longer R6.1
- net Supply: now also R4.2; no longer R4.1
- net VBUSF: now also R4.1; no longer R4.2

Commit message: updated:   Hardware/KiCad9/cloudSmoker_ver2f.kicad_pcb
Other:
- note removed: "check TP8 is this correct?"
Changed lines of the file:
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@@
-		)
-	)
-	(text "check TP8 is this correct?\n"
-		(exclude_from_sim no)
-		(at 213.36 131.064 0)
-		(effects
-			(font
-				(size 1 1)
-				(italic yes)
-				(color 255 0 0 1)
-			)
 		)
 	)
