File: Hardware/KiCad9/cloudSmoker_ver2f.kicad_sch (KiCad schematic)
At the start: 98 parts, among them J1 Conn_01x02_Pin, J10 Conn_01x04_Pin, J11 Conn_01x04_Pin, J12 AudioJack2_SwitchT, J13 AudioJack2_SwitchT, J14 Conn_01x04_Pin, J15 Conn_01x04_Pin, J16 AudioJack2_SwitchT, J2 Conn_01x04_Socket, J3 Conn_01x04_Pin, J4 Conn_01x08, J5 Conn_01x04_Socket, J6 Conn_01x04_Pin, J7 Conn_01x05, J8 Conn_01x05_Socket, J9 AudioJack2_SwitchT, Q1 BSS138, Q2 BSS138, SW1 RotaryEncoder_Switch, SW2 SW_Push_Dual, SW3 SW_Push_Dual, U1 TLV76733DGNR, U2 INA226AIDGSR, U3 GT-USB-7010ASV, U4 ESP32-C3-WROOM-02U-N4, U5 SRV05-4-P-T7, U6 ADS1115IRUGR, U7 SRV05-4-P-T7

Commit message: update files
Other:
- note added: "Ground shunt to use for probe insert detection"
Changed lines of the file:
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@@
+		)
+	)
+	(text "Ground shunt to use for probe insert detection"
+		(exclude_from_sim yes)
+		(at 59.182 175.768 0)
+		(effects
+			(font
+				(face "KiCad Font")
+				(size 1 1)
+			)
 		)
 	)

Commit message: fixed schematic text note errors
Other:
- note added: "Display module has integrated transistor for Backlight control 3V3 logic signal safe (no level shifting required)"
- note removed: "Display module has integrated transistor for Backlight control 3V3 logic signal safe"
Changed lines of the file:
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@@
 		)
 	)
-	(text "Display module has integrated \ntransistor for Backlight control\n\n3V3 logic signal safe\n"
+	(text "Display module has integrated \ntransistor for Backlight control\n\n3V3 logic signal safe (no level shifting required)\n"
 		(exclude_from_sim no)
 		(at 378.968 80.264 0)
@@
 		(row_heights 2.54 2.54 2.54 2.54 2.54)
 		(cells
-			(table_cell "5V"
+			(table_cell "3V3"
 				(exclude_from_sim no)
 				(at 358.394 115.57 0)
@@
 				)
 			)
-			(table_cell "+5V"
+			(table_cell "+3.3V"
 				(exclude_from_sim no)
 				(at 383.794 115.57 0)
