File: Hardware/KiCad9/cloudSmoker_ver2f.kicad_pcb (KiCad board)
At the start: 4 copper layers, 70 x 70 mm, 115 parts, among them J1 Conn_01x02_Pin, J11 Conn_01x04_Pin, J15 Conn_01x04_Pin, J3 Conn_01x04_Pin, J6 Conn_01x04_Pin, J7 Conn_01x05, Q1 BSS138, Q2 BSS138, SW2 SW_Push_Dual, SW3 SW_Push_Dual, U1 TLV76733DGNR, U2 INA226AIDGSR, U3 GT-USB-7010ASV, U4 ESP32-C3-WROOM-02U-N4, U5 SRV05-4-P-T7, U6 ADS1115IRUGR, U7 SRV05-4-P-T7

Commit message: updated gitigner, added enclosure files, added new images, added new step file for pcb
Parts:
- U1: value TLV76733DGNR -> ~
- U2: value INA226AIDGSR -> ~
- U5, U7: value SRV05-4-P-T7 -> ~
- U6: value ADS1115IRUGR -> ~
